Commit message: fix: Add spring to suspension joints to keep body level

File: urdf/rover.urdf.xacro (robot description, xacro)
@@ -61,6 +61,6 @@
     <child link="Sag_suspansiyon_merkezi" />
     <axis xyz="0 1 0" />
-    <limit lower="-0.5236" upper="0.5236" effort="100" velocity="1.0" />
-    <dynamics damping="10.0" friction="1.0"/>
+    <limit lower="-0.3" upper="0.3" effort="100" velocity="1.0" />
+    <dynamics damping="5.0" friction="1.0"/>
   </joint>
   <link name="right_front_wheel">
@@ -153,6 +153,6 @@
     <child link="Sol_Suspensiyon_merkezi" />
     <axis xyz="0 1 0" />
-    <limit lower="-0.5236" upper="0.5236" effort="100" velocity="1.0" />
-    <dynamics damping="10.0" friction="1.0"/>
+    <limit lower="-0.3" upper="0.3" effort="100" velocity="1.0" />
+    <dynamics damping="5.0" friction="1.0"/>
   </joint>
   <link name="left_front_wheel">
@@ -252,4 +252,13 @@
     <minDepth>0.001</minDepth>
     <maxVel>1.0</maxVel>
+  </gazebo>
+  <!-- Süspansiyon Spring Parametreleri -->
+  <gazebo reference="Sag_Suspansiyon_merkezi_joint">
+    <springStiffness>500</springStiffness>
+    <springReference>0</springReference>
+  </gazebo>
+  <gazebo reference="Sol_Suspensiyon_merkezi_joint">
+    <springStiffness>500</springStiffness>
+    <springReference>0</springReference>
   </gazebo>
   <!-- ===================== ROS2 CONTROL ===================== -->

Commit message: Feat : Robotics arm added

File: urdf/rover.urdf.xacro (robot description, xacro)
@@ -1,4 +1,6 @@
 <?xml version="1.0" encoding="utf-8"?>
 <robot name="rover" xmlns:xacro="http://www.ros.org/wiki/xacro">
+  <!-- Include Robotic Arm -->
+  <xacro:include filename="$(find rover_sim)/urdf/arm.urdf.xacro" />
   <!-- Include original URDF structure -->
   <link name="base_link">
@@ -303,4 +305,50 @@
       <state_interface name="velocity"/>
     </joint>
+    <!-- ========== ARM JOINTS ========== -->
+    <!-- Arm Joint 1 - Base rotation -->
+    <joint name="arm_joint1">
+      <command_interface name="position">
+        <param name="min">-3.14159</param>
+        <param name="max">3.14159</param>
+      </command_interface>
+      <state_interface name="position"/>
+      <state_interface name="velocity"/>
+    </joint>
+    <!-- Arm Joint 2 - Shoulder -->
+    <joint name="arm_joint2">
+      <command_interface name="position">
+        <param name="min">-1.57</param>
+        <param name="max">1.57</param>
+      </command_interface>
+      <state_interface name="position"/>
+      <state_interface name="velocity"/>
+    </joint>
+    <!-- Arm Joint 3 - Elbow -->
+    <joint name="arm_joint3">
+      <command_interface name="position">
+        <param name="min">-2.0</param>
+        <param name="max">2.0</param>
+      </command_interface>
+      <state_interface name="position"/>
+      <state_interface name="velocity"/>
+    </joint>
+    <!-- Arm Joint 4 - Wrist pitch -->
+    <joint name="arm_joint4">
+      <command_interface name="position">
+        <param name="min">-2.0</param>
+        <param name="max">2.0</param>
+      </command_interface>
+      <state_interface name="position"/>
+      <state_interface name="velocity"/>
+    </joint>
+    <!-- Arm Joint 5 - Wrist roll -->
+    <joint name="arm_joint5">
+      <command_interface name="position">
+        <param name="min">-3.14159</param>
+        <param name="max">3.14159</param>
+      </command_interface>
+      <state_interface name="position"/>
+      <state_interface name="velocity"/>
+    </joint>
   </ros2_control>
   <!-- Gazebo plugin for ros2_control -->

Commit message: fix: Turning and brake paramaters was updated

File: urdf/rover.urdf.xacro (robot description, xacro)
@@ -64,5 +64,5 @@
     <axis xyz="0 1 0" />
     <limit lower="-0.3" upper="0.3" effort="100" velocity="1.0" />
-    <dynamics damping="5.0" friction="1.0"/>
+    <dynamics damping="1.5" friction="0.5"/>
   </joint>
   <link name="right_front_wheel">
@@ -156,5 +156,5 @@
     <axis xyz="0 1 0" />
     <limit lower="-0.3" upper="0.3" effort="100" velocity="1.0" />
-    <dynamics damping="5.0" friction="1.0"/>
+    <dynamics damping="1.5" friction="0.5"/>
   </joint>
   <link name="left_front_wheel">
@@ -182,5 +182,5 @@
   </link>
   <joint name="left_front_wheel_joint" type="continuous">
-    <origin xyz="0.52892 0.1827 -0.30434" rpy="0 0 0" />
+    <origin xyz="0.51315 0.1837 -0.33036" rpy="0 0 0" />
     <parent link="Sol_Suspensiyon_merkezi" />
     <child link="left_front_wheel" />
@@ -212,5 +212,5 @@
   </link>
   <joint name="left_rear_wheel_joint" type="continuous">
-    <origin xyz="-0.54459 0.1827 -0.27547" rpy="0 0 0" />
+    <origin xyz="-0.55762 0.1827 -0.24797" rpy="0 0 0" />
     <parent link="Sol_Suspensiyon_merkezi" />
     <child link="left_rear_wheel" />

Commit message: Feat: Camera gui module added

File: urdf/rover.urdf.xacro (robot description, xacro)
@@ -120,5 +120,5 @@
   </link>
   <joint name="right_rear_wheel_joint" type="continuous">
-    <origin xyz="-0.55762 -0.1827 -0.24797" rpy="0 0 0" />
+    <origin xyz="-0.55762 -0.1827 -0.33036" rpy="0 0 0" />
     <parent link="Sag_suspansiyon_merkezi" />
     <child link="right_rear_wheel" />
@@ -212,5 +212,5 @@
   </link>
   <joint name="left_rear_wheel_joint" type="continuous">
-    <origin xyz="-0.55762 0.1827 -0.24797" rpy="0 0 0" />
+    <origin xyz="-0.55762 0.1827 -0.33036" rpy="0 0 0" />
     <parent link="Sol_Suspensiyon_merkezi" />
     <child link="left_rear_wheel" />
@@ -352,4 +352,58 @@
     </joint>
   </ros2_control>
+  <!-- ===================== CAMERA ===================== -->
+  <!-- Camera Link -->
+  <link name="camera_link">
+    <inertial>
+      <origin xyz="0 0 0" rpy="0 0 0" />
+      <mass value="0.05" />
+      <inertia ixx="0.0001" ixy="0.0" ixz="0.0"
+               iyy="0.0001" iyz="0.0" izz="0.0001" />
+    </inertial>
+    <visual>
+      <origin xyz="0 0 0" rpy="0 0 0" />
+      <geometry>
+        <box size="0.03 0.05 0.02"/>
+      </geometry>
+      <material name="camera_blue">
+        <color rgba="0.2 0.2 0.8 1" />
+      </material>
+    </visual>
+    <collision>
+      <origin xyz="0 0 0" rpy="0 0 0" />
+      <geometry>
+        <box size="0.03 0.05 0.02"/>
+      </geometry>
+    </collision>
+  </link>
+  <!-- Camera Joint - Rover'ın ön tarafına monte -->
+  <joint name="camera_joint" type="fixed">
+    <origin xyz="0.25 0 0.05" rpy="0 0 0" />
+    <parent link="base_link" />
+    <child link="camera_link" />
+  </joint>
+  <!-- Gazebo Camera Sensor -->
+  <gazebo reference="camera_link">
+    <sensor name="camera_sensor" type="camera">
+      <pose>0 0 0 0 0 0</pose>
+      <update_rate>30</update_rate>
+      <always_on>1</always_on>
+      <visualize>true</visualize>
+      <topic>/rover/camera/image_raw</topic>
+      <camera name="rover_camera">
+        <horizontal_fov>1.047</horizontal_fov>
+        <image>
+          <width>640</width>
+          <height>480</height>
+          <format>R8G8B8</format>
+        </image>
+        <clip>
+          <near>0.05</near>
+          <far>100.0</far>
+        </clip>
+      </camera>
+    </sensor>
+    <material>Gazebo/Blue</material>
+  </gazebo>
   <!-- Gazebo plugin for ros2_control -->
   <gazebo>
